File: ARM7TDMIBreakout.sch (KiCad schematic (older format))
At the start: 8 parts, among them J1 Conn_01x24_MountingPin_24-1, J2 Conn_01x24_MountingPin_48-1, U1 ARM7TDMI

Commit message: Fixed: Connected bypass capacitors to AGND
Connections:
- net GND: now also J1.23 (Pin_23), U1.23 (AGND)
Changed lines of the file:
@@
 	19350 13350 19350 13950
 Wire Wire Line
-	18275 17800 21225 17800
+	18275 17800 20300 17800
 Wire Wire Line
 	21225 14800 21225 14725
@@
 L power:PWR_FLAG #FLG0102
 U 1 1 5DC8510F
-P 21225 17800
-F 0 "#FLG0102" H 21225 17875 50  0001 C CNN
-F 1 "PWR_FLAG" H 21225 17973 50  0000 C CNN
-F 2 "" H 21225 17800 50  0001 C CNN
-F 3 "~" H 21225 17800 50  0001 C CNN
-	1    21225 17800
+P 20300 17800
+F 0 "#FLG0102" H 20300 17875 50  0001 C CNN
+F 1 "PWR_FLAG" H 20300 17973 50  0000 C CNN
+F 2 "" H 20300 17800 50  0001 C CNN
+F 3 "~" H 20300 17800 50  0001 C CNN
+	1    20300 17800
 	-1   0    0    1
 $EndComp
@@
 $EndComp
 Connection ~ 25225 17100
-Connection ~ 21225 17800
 $Comp
 L power:PWR_FLAG #FLG0103
@@
 Text Label 20900 13100 1    50   ~ 0
 P1.1
+$Comp
+L power:GND #PWR?
+U 1 1 5DCEFA76
+P 20900 17800
+F 0 "#PWR?" H 20900 17550 50  0001 C CNN
+F 1 "GND" H 20905 17627 50  0000 C CNN
+F 2 "" H 20900 17800 50  0001 C CNN
+F 3 "" H 20900 17800 50  0001 C CNN
+	1    20900 17800
+	1    0    0    -1
+$EndComp
+Connection ~ 20300 17800
+Wire Wire Line
+	20300 17800 20900 17800
+Connection ~ 20900 17800
+Wire Wire Line
+	20900 17800 21225 17800
 $EndSCHEMATC
